Commit message: Updating URDF and meshes

File: pfields_demo/urdf/fer_franka_hand.urdf (robot description, URDF)
Before this commit: robot fer, 23 links, 22 joints
Links:
- link fer_hand: geometry collision mesh filename=package://pfields_demo/meshes/robot_ee/franka_hand_white/co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; visual mesh filename=package://pfields_demo/meshes/robot_ee/franka_hand_white/vi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
- link fer_leftfinger: geometry collision box size=17.5e-3 15.2e-3 18.5e-3; collision box size=17.5e-3 7e-3 23.5e-3
- link fer_link0: geometry collision mesh filename=package://pfields_demo/meshes/robot_arms/fer/collision/link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; visual mesh filename=package://pfields_demo/meshes/robot_arms/fer/visual/link0.d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
- link fer_link1: geometry collision mesh filename=package://pfields_demo/meshes/robot_arms/fer/collision/link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; visual mesh filename=package://pfields_demo/meshes/robot_arms/fer/visual/link1.d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
- link fer_link2: geometry collision mesh filename=package://pfields_demo/meshes/robot_arms/fer/collision/link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; visual mesh filename=package://pfields_demo/meshes/robot_arms/fer/visual/link2.d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
- link fer_link3: geometry collision mesh filename=package://pfields_demo/meshes/robot_arms/fer/collision/link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; visual mesh filename=package://pfields_demo/meshes/robot_arms/fer/visual/link3.d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
- link fer_link4: geometry collision mesh filename=package://pfields_demo/meshes/robot_arms/fer/collision/link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; visual mesh filename=package://pfields_demo/meshes/robot_arms/fer/visual/link4.d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
- link fer_link5: geometry collision mesh filename=package://pfields_demo/meshes/robot_arms/fer/collision/link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; visual mesh filename=package://pfields_demo/meshes/robot_arms/fer/visual/link5.d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
- link fer_link6: geometry collision mesh filename=package://pfields_demo/meshes/robot_arms/fer/collision/link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; visual mesh filename=package://pfields_demo/meshes/robot_arms/fer/visual/link6.d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
- link fer_link7: geometry collision mesh filename=package://pfields_demo/meshes/robot_arms/fer/collision/link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; visual mesh filename=package://pfields_demo/meshes/robot_arms/fer/visual/link7.d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
- link fer_rightfinger: geometry collision box size=17.5e-3 15.2e-3 18.5e-3; collision box size=17.5e-3 7e-3 23.5e-3
