Commit message: pfields_demo -> potential_fields_demos

File: potential_fields_demos/urdf/fer_franka_hand.urdf (robot description, URDF)
Before this commit: robot fer, 23 links, 22 joints
Links:
- link fer_hand: geometry collision mesh filename=package://potential_fields_demos/meshes/robot_ee/franka_han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; visual mesh filename=package://potential_fields_demos/meshes/robot_ee/franka_han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
- link fer_leftfinger: geometry collision box size=17.5e-3 15.2e-3 18.5e-3; collision box size=17.5e-3 7e-3 23.5e-3
- link fer_link0: geometry collision mesh filename=package://potential_fields_demos/meshes/robot_arms/fer/coll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; visual mesh filename=package://potential_fields_demos/meshes/robot_arms/fer/visu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
- link fer_link1: geometry collision mesh filename=package://potential_fields_demos/meshes/robot_arms/fer/coll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; visual mesh filename=package://potential_fields_demos/meshes/robot_arms/fer/visu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
- link fer_link2: geometry collision mesh filename=package://potential_fields_demos/meshes/robot_arms/fer/coll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; visual mesh filename=package://potential_fields_demos/meshes/robot_arms/fer/visu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
- link fer_link3: geometry collision mesh filename=package://potential_fields_demos/meshes/robot_arms/fer/coll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; visual mesh filename=package://potential_fields_demos/meshes/robot_arms/fer/visu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
- link fer_link4: geometry collision mesh filename=package://potential_fields_demos/meshes/robot_arms/fer/coll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; visual mesh filename=package://potential_fields_demos/meshes/robot_arms/fer/visu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
- link fer_link5: geometry collision mesh filename=package://potential_fields_demos/meshes/robot_arms/fer/coll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; visual mesh filename=package://potential_fields_demos/meshes/robot_arms/fer/visu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
- link fer_link6: geometry collision mesh filename=package://potential_fields_demos/meshes/robot_arms/fer/coll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; visual mesh filename=package://potential_fields_demos/meshes/robot_arms/fer/visu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
- link fer_link7: geometry collision mesh filename=package://potential_fields_demos/meshes/robot_arms/fer/coll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; visual mesh filename=package://potential_fields_demos/meshes/robot_arms/fer/visu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
- link fer_rightfinger: geometry collision box size=17.5e-3 15.2e-3 18.5e-3; collision box size=17.5e-3 7e-3 23.5e-3

File: potential_fields_demos/urdf/xarm7.urdf (robot description, URDF)
Before this commit: robot UF_ROBOT, 10 links, 9 joints
Links:
- link link1: geometry collision mesh filename=package://potential_fields_demos/meshes/xarm7/visual/link1.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; visual mesh filename=package://potential_fields_demos/meshes/xarm7/visual/link1.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
- link link2: geometry collision mesh filename=package://potential_fields_demos/meshes/xarm7/visual/link2.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; visual mesh filename=package://potential_fields_demos/meshes/xarm7/visual/link2.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
- link link3: geometry collision mesh filename=package://potential_fields_demos/meshes/xarm7/visual/link3.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; visual mesh filename=package://potential_fields_demos/meshes/xarm7/visual/link3.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
- link link4: geometry collision mesh filename=package://potential_fields_demos/meshes/xarm7/visual/link4.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; visual mesh filename=package://potential_fields_demos/meshes/xarm7/visual/link4.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
- link link5: geometry collision mesh filename=package://potential_fields_demos/meshes/xarm7/visual/link5.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; visual mesh filename=package://potential_fields_demos/meshes/xarm7/visual/link5.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
- link link6: geometry collision mesh filename=package://potential_fields_demos/meshes/xarm7/visual/link6.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; visual mesh filename=package://potential_fields_demos/meshes/xarm7/visual/link6.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
- link link7: geometry collision mesh filename=package://potential_fields_demos/meshes/xarm7/visual/link7.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; visual mesh filename=package://potential_fields_demos/meshes/xarm7/visual/link7.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
- link link_base: geometry collision mesh filename=package://potential_fields_demos/meshes/xarm7/visual/link_b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; visual mesh filename=package://potential_fields_demos/meshes/xarm7/visual/link_b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
